Commit message: update chapter8_1 joints_state

File: learning/chapter8_1/src/robot_description/urdf/robot_base.urdf (robot description, URDF)
Before this commit: robot robot, 2 links, 1 joints
Links:
- added link base_footprint
- added link caster_link; visual sphere radius=0.016
- added link imu_link; visual box size=0.02 0.02 0.02
- added link left_wheel_link; visual cylinder length=0.04 radius=0.032
- added link right_wheel_link; visual cylinder length=0.04 radius=0.032
Joints:
- added joint base_joint: type fixed, parent base_footprint, child base_link, origin xyz=0.0 0.0 0.076 rpy=0 0 0
- added joint caster_joint: type fixed, parent base_link, child caster_link, origin xyz=0.06 0.0 -0.076
- added joint imu_joint: type fixed, parent base_link, child imu_link, origin xyz=0 0 0.02
- added joint left_wheel_joint: type continuous, parent base_link, child left_wheel_link, origin xyz=-0.02 0.10 -0.06, axis 0 1 0
- added joint right_wheel_joint: type continuous, parent base_link, child right_wheel_link, origin xyz=-0.02 -0.10 -0.06, axis 0 1 0
